File: PCB/IMU_node/imu_node.sch (EAGLE design)
At the start: 40 parts, among them IC1 MCP73831/OT, IC2 BN055, J1 LiPo Battery, J2 UART_Interface, J3 ISP_Interface, SW1 Reset, SW2 Bootloader, U1 32U4, U2 MAX1704X

Commit message: Added latest version of IMU node PCB
Parts:
- added C10, C14, C15: 100nF, ipc-7351-capacitor:CAPACITOR_0603
- added C11: 10µF, ipc-7351-capacitor:CAPACITOR_0603
- added C12, C13, C8, C9: 22pF, ipc-7351-capacitor:CAPACITOR_0603
- added R15, R16, R17, R18: 10k, ipc-7351-resistor:RESISTOR_0603
- added Y1: 32.768kHz, SparkFun-Clocks:CRYSTAL-32.768KHZSMD-3.2X1.5
- added Y4: 8MHz, SparkFun-Clocks:CRYSTAL-8MHZSMD-5X3.2
- R4, R5: value (none) -> 470
- U$2: value 6-PIN-BREAKOUT6-PIN-BREAKOUT -> nRF24L01+
Connections:
- net PCINT6_BAT_ALERT renamed PCINT6
- removed net PD0_SCL: R11.2, U1.PD0(SCL), U2.SCL
- removed net PD1_SDA: R10.2, U1.PD1(SDA), U2.SDA
- new net !HWB!: R16.2, SW2.P, SW2.P1, U1.PE2/!HWB
- new net !RESET!: J3.5, R15.2, SW1.P, SW1.P1, U1.!RESET
- new net CE: U$2.CE, U1.PB5(ADC12)
- new net INT6: U$2.IRQ, U1.PE6
- new net MISO: J3.1, U$2.MISO, U1.PB3(MISO)
- new net MOSI: J3.4, U$2.MOSI, U1.PB2(MOSI)
- new net N$10: C9.1, U1.XTAL1, Y4.2
- new net N$11: C8.1, U1.XTAL2, Y4.1
- new net N$12: C10.1, U1.AREF
- new net N$15: LED4.A, R5.1
- new net N$16: C12.2, IC2.XOUT32, Y1.2
- new net N$17: LED5.A, R4.1
- new net N$19: IC2.RESET, R17.2
- new net N$20: C15.1, IC2.CAP
- new net N$21: IC2.BOOT_MODE_SEL, R18.2
- new net OC3A: R5.2, U1.PC6
- new net OC4A: R4.2, U1.PC7
- new net PCINT4: IC2.INT_OUT, U1.PB4(ADC11)
- new net SCK: J3.3, U$2.SCK, U1.PB1(SCK)
- new net SCL: IC2.COM1-SCL, R11.2, U1.PD0(SCL), U2.SCL
- new net SDA: IC2.COM0-SDA, R10.2, U1.PD1(SDA), U2.SDA
- new net SS: U$2.!CSN!, U1.PB0(SS)
- new net UART_RX: J2.1, U1.PD2(RX)
- new net UART_TX: J2.2, U1.PD3(TX)
- net +3V3: now also C11.1, C14.1, IC2.VDD, IC2.VDDIO, J3.2, R15.1, R16.1, R17.1, R18.1, U$2.VCC, U1.AVCC@24, U1.AVCC@44, U1.UCAP, U1.VCC@14, U1.VCC@34
- net GND: now also C10.2, C11.2, C12.1, C13.2, C14.2, C15.2, C8.2, C9.2, IC2.COM2, IC2.COM3-SA0, IC2.GND, IC2.GND_IO, IC2.PIN10, IC2.PIN15, IC2.PIN16, IC2.PS0, IC2.PS1, J2.3, J3.6, LED4.C, LED5.C, SW1.S, SW1.S1, SW2.S, SW2.S1, U$2.GND, U1.GND@15, U1.GND@23, U1.GND@35, U1.GND@43, U1.UGND
- net N$6: now also C13.1, IC2.XIN32, Y1.1; no longer U1.UVCC
Other:
- note added: "0x28"
- note added: "Input-Output Unit (IOU)"
- note added: "Program-Debug Unit (PDU)"
- note added: "nRF24L01+"
- moved on the sheet: CN1, IC2, J1, J2, J3, LED4, LED5, R4, R5, R6, R7, SW1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
