File: PCB/IMU_node/imu_node.brd (EAGLE design)
At the start: 45 x 29.8 mm, 40 parts, among them IC1 MCP73831/OT, IC2 BN055, J1 LiPo Battery, J2 UART_Interface, J3 ISP_Interface, SW1 Reset, SW2 Bootloader, U1 32U4, U2 MAX1704X

Commit message: Added latest version of IMU node PCB
Parts:
- added C10, C14, C15: 100nF, ipc-7351-capacitor:CAPC1608X92N
- added C11: 10µF, ipc-7351-capacitor:CAPC1608X92N
- added C12, C13, C8, C9: 22pF, ipc-7351-capacitor:CAPC1608X92N
- added R15, R16, R17, R18: 10k, ipc-7351-resistor:RESC1608X55N
- added Y1: 32.768kHz, SparkFun-Clocks:CRYSTAL-SMD-3.2X1.5MM
- added Y4: 8MHz, SparkFun-Clocks:CRYSTAL-SMD-5X3.2-4PAD
- R4, R5: value (none) -> 470
- U$2: value 6-PIN-BREAKOUT6-PIN-BREAKOUT -> nRF24L01+
- moved SW2 116.7 mm to (-17.7, 15.4)
- moved IC2 45.6 mm to (18.5, 44.6)
Connections:
- net PCINT6_BAT_ALERT renamed PCINT6
- removed net GND_IO: IC2.25
- removed net PD0_SCL: R11.2, U1.18, U2.7
- removed net PD1_SDA: R10.2, U1.19, U2.8
- removed net VDD: IC2.3
- removed net VDDIO: IC2.28
- new net !HWB!: R16.2, SW2.1, SW2.3, U1.33
- new net !RESET!: J3.5, R15.2, SW1.1, SW1.3, U1.13
- new net CE: U$2.2, U1.29
- new net INT6: U$2.7, U1.1
- new net MISO: J3.1, U$2.6, U1.11
- new net MOSI: J3.4, U$2.5, U1.10
- new net N$10: C9.1, U1.17, Y4.3
- new net N$11: C8.1, U1.16, Y4.1
- new net N$12: C10.1, U1.42
- new net N$15: LED4.A, R5.1
- new net N$16: C12.2, IC2.26, Y1.P$2
- new net N$17: LED5.A, R4.1
- new net N$19: IC2.11, R17.2
- new net N$20: C15.1, IC2.9
- new net N$21: IC2.4, R18.2
- new net OC3A: R5.2, U1.31
- new net OC4A: R4.2, U1.32
- new net PCINT4: IC2.14, U1.28
- new net SCK: J3.3, U$2.4, U1.9
- new net SCL: IC2.19, R11.2, U1.18, U2.7
- new net SDA: IC2.20, R10.2, U1.19, U2.8
- new net SS: U$2.3, U1.8
- new net UART_RX: J2.1, U1.20
- new net UART_TX: J2.2, U1.21
- net +3V3: now also C11.1, C14.1, IC2.28, IC2.3, J3.2, R15.1, R16.1, R17.1, R18.1, U$2.1, U1.14, U1.24, U1.34, U1.44, U1.6
- net GND: now also C10.2, C11.2, C12.1, C13.2, C14.2, C15.2, C8.2, C9.2, IC2.10, IC2.15, IC2.16, IC2.17, IC2.18, IC2.25, IC2.5, IC2.6, J2.3, J3.6, LED4.C, LED5.C, SW1.2, SW1.4, SW2.2, SW2.4, U$2.8, U1.15, U1.23, U1.35, U1.43, U1.5
- net N$6: now also C13.1, IC2.27, Y1.P$1; no longer U1.2

Commit message: Added the first version of IMU_node, IMU_finger & IMU_hand PCBs
Parts:
- removed J1: LiPo Battery, SparkFun-Connectors:JST-2-SMD
- added J4: BAT_CON, SparkFun-Connectors:1X02
- CN1: value (none) -> USB_CON
- moved R18 257.3 mm to (39.2, 24.3), turned to 90 degrees
- moved R17 255.6 mm to (39.2, 27.6), turned to 90 degrees
- moved C15 252.2 mm to (41.0, 27.6), turned to 270 degrees
- moved C14 245.2 mm to (41.0, 24.3), turned to 270 degrees
- moved C13 236.6 mm to (37.8, 21.1), turned to 270 degrees
- moved C12 229.1 mm to (32.1, 21.1), turned to 90 degrees
- moved Y1 227.4 mm to (34.9, 21.9), turned to 180 degrees
- moved C11 203.6 mm to (19.1, 7.10), turned to 270 degrees
- moved C9 202.8 mm to (32.1, 17.6), turned to 270 degrees
- moved C8 202.5 mm to (37.8, 17.5), turned to 90 degrees
- moved C10 198.3 mm to (17.3, 7.10), turned to 270 degrees
- moved R15 197.7 mm to (35.0, 3.20), turned to 90 degrees
- moved R16 197.6 mm to (28.5, 3.17), turned to 90 degrees
- moved C7 182.8 mm to (6.55, 26.8), turned to 90 degrees
- moved R14 179.8 mm to (2.24, 20.8), turned to 180 degrees
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Connections:
- net GND: now also J4.1; no longer J1.1
- net VBAT: now also J4.2; no longer J1.2
Routing:
- net +3V3: track 0.00 -> 148.2 mm, vias 0 -> 4
- net !RESET!: track 0.00 -> 46.6 mm, vias 0 -> 2
- net VBUS: track 0.00 -> 41.4 mm, vias 0 -> 4
- net VBUS_RAW: track 0.00 -> 37.3 mm, vias 0 -> 3
- net VBAT: track 0.00 -> 33.7 mm, vias 0 -> 1
- net SDA: track 0.00 -> 30.6 mm, vias 0 -> 3
- net SCK: track 0.00 -> 29.0 mm
- net !HWB!: track 0.00 -> 27.7 mm, vias 0 -> 2
- net SCL: track 0.00 -> 25.6 mm, vias 0 -> 2
- net MOSI: track 0.00 -> 21.7 mm
- net INT6: track 0.00 -> 21.5 mm
- net MISO: track 0.00 -> 21.2 mm
- net CE: track 0.00 -> 19.5 mm, vias 0 -> 1
- net PCINT4: track 0.00 -> 19.0 mm, vias 0 -> 2
- net N$11: track 0.00 -> 18.7 mm, vias 0 -> 2
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- added copper zone on layer 1, net GND
- added copper zone on layer 16, net GND
