File: PCB/IMU_hand/imu_hand.sch (EAGLE design)
At the start: 54 parts, among them CN1 USB_CON, IC1 MCP73831/OT, IC2 BN055, J2 UART_Interface, J3 ISP_Interface, J4 BAT_CON, SW1 Reset, SW2 Bootloader, U1 32U4, U2 MAX1704X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

Commit message: Added the first version of IMU_node, IMU_finger & IMU_hand PCBs
Parts:
- removed R8: 100k, ipc-7351-resistor:RESISTOR_0603
- removed U$1: SPX3819_3.3, SparkFun-IC-Power:V_REG_SPX3819-SOT23-5
- added C16: (no value), ipc-7351-capacitor:CAPACITOR_0603
- added IC3: 74HC4051D, 74HC4051D:74HC4051D
- added J1, J5, J6, J7, J8: (no value), SparkFun-Connectors:CONN_04SMD2
- added R19: 10k, ipc-7351-resistor:RESISTOR_0603
- added U4: Value, TPS79633-Q1:TPS79633QDCQRQ1
- C1: value 10µF -> 2.2µF
- C2: value 1µF -> 0.01µF
- C3: value 10µF -> 1µF
- J2: device SparkFun-Connectors:CONN_03 -> SparkFun-Connectors:CONN_02
- S1: device SparkFun-Switches:SWITCH-SPDT-SMD-RIGHT-ANGLE -> SparkFun-Switches:SWITCH-SPDT-PTH-11.6X4.0MM
Connections:
- new net N$18: IC3.Y4, J1.2
- new net N$22: IC3.Y2, J5.2
- new net N$23: IC3.Y1, J6.2
- new net N$24: IC3.Y0, J7.2
- new net N$25: IC3.Y3, J8.2
- new net N$26: IC3.!E, R19.2
- new net S0: IC3.S0, U1.PD4(ADC8)
- new net S1: IC3.S1, U1.PD6(ADC9)
- new net S2: IC3.S2, U1.PD7(ADC10)
- new net Y5_SDA: IC2.COM0-SDA, IC3.Y5
- net +3V3: now also C16.2, IC3.VCC, J1.1, J5.1, J6.1, J7.1, J8.1, U4.OUT; no longer C2.2, U$1.OUT
- net GND: now also C16.1, IC3.GND, IC3.VEE, J1.4, J5.4, J6.4, J7.4, J8.4, R19.1, U4.GND, U4.GND_2; no longer J2.3, U$1.GND
- net N$5: now also C2.2, U4.NR_FB; no longer R8.2, U$1.EN
- net SCL: now also J1.3, J5.3, J6.3, J7.3, J8.3
- net SDA: now also IC3.Z; no longer IC2.COM0-SDA
- net VBUS: now also U4.EN, U4.IN; no longer R8.1, U$1.IN
Other:
- note added: "Mux-Demux Unit (MDU)"
